File: hardware/reva/reva.sch (KiCad schematic (older format))
At the start: 22 parts, among them U1 ATSAMD21E17D-A, U2 DRV8833PWP, U3 MIC5504-3.3YM5, Y1 Crystal

Commit message: schema update
Parts:
- added C1: 10u 16V, Capacitor_SMD:C_0603_1608Metric, symbol Device:C
- added C10, C4: 10u 10V, Capacitor_SMD:C_0603_1608Metric, symbol Device:C
- added C11, C9: 100n, Capacitor_SMD:C_0603_1608Metric, symbol Device:C
- added C12: 10n, Capacitor_SMD:C_0603_1608Metric, symbol Device:C
- added C13: 2u2, Capacitor_SMD:C_0603_1608Metric, symbol Device:C
- added C8: 1u 25V, Capacitor_SMD:C_0603_1608Metric, symbol Device:C
- added D1, D7: D_Schottky, Diode_SMD:D_SMA, symbol Device:D_Schottky
- added D2, D3, D4, D5: LED, LED_SMD:LED_0603_1608Metric, symbol Device:LED
- added FB2: BLM18PG471SZ1D, Inductor_SMD:L_0603_1608Metric, symbol Device:FerriteBead
- added J2: Conn_01x05, symbol Connector_Generic:Conn_01x05
- added R1, R16, R17, R18, R2, R4, R6: 10k, Resistor_SMD:R_0603_1608Metric, symbol Device:R
- added R10, R7, R8, R9: 330, Resistor_SMD:R_0603_1608Metric, symbol Device:R
- added R14, R15: R, Resistor_SMD:R_0603_1608Metric, symbol Device:R
- added SW1: Mode, symbol Switch:SW_Push
- added SW2: Up, symbol Switch:SW_Push
- added SW3: Down, symbol Switch:SW_Push
- added SW4: Sel, symbol Switch:SW_Push
- added SW5: Reset, symbol Switch:SW_Push
- C2, C3, C5, C6: renamed from C?; footprint (none) -> Capacitor_SMD:C_0603_1608Metric
- C7: renamed from C?; value C -> 10n; footprint (none) -> Capacitor_SMD:C_0603_1608Metric
- FB1: renamed from FB?; footprint (none) -> Inductor_SMD:L_0603_1608Metric
- R11, R12, R3, R5: renamed from R?; footprint (none) -> Resistor_SMD:R_0603_1608Metric
- R13: renamed from R?; value R -> 330; footprint (none) -> Resistor_SMD:R_0603_1608Metric
- gave numbers to parts that had none: 2
Connections:
- net EXT_RES: now also SW5.2
- net GND: now also D6.1 (GND), J1.3 (Pin_3), J1.5 (Pin_5), U1.10 (GND), U1.28 (GND), U2.13 (GND), U2.17 (GND(PPAD)), U3.2 (GND), USB1.13 (SHIELD), C1.2, C10.2, C11.2, C13.1, C4.2, C8.2, C9.2, R14.2, R15.2, SW1.1, SW2.1, SW3.1, SW4.1, SW5.1
- net RESET: now also J1.10 (Pin_10), R16.2
- net SWCLK: now also J1.2 (Pin_2), R17.2
- net SWDIO: now also J1.4 (Pin_4)
- net USART_RX: now also J1.7 (Pin_7)
- net USART_TX: now also J1.9 (Pin_9)
- net VBUS: now also D1.2 (A)
- net SW_Sel: now reaches U1.16 (PA15)
- net SW_Sel: now also J1.8 (Pin_8), R6.2, SW4.2
- net at U1.29 (VDDCORE): now also C8.1
- net +3V3: now reaches U1.30 (VDDIN)
- net +3V3: now also J1.1 (Pin_1), U3.5 (VOUT), C11.1, C4.1, C9.1, FB2.1, R1.1, R10.2, R16.1, R17.1, R18.1, R2.1, R4.1, R6.1, R7.2, R8.2, R9.2
- net at U1.9 (VDDANA): now also C10.1, FB2.2
- net nSleep: now reaches U2.1 (nSLEEP)
- net BIN2: now reaches U2.10 (BIN2)
- net at U2.11 (VCP): now also C12.1
- net VDC: now reaches U2.12 (VM)
- net VDC: now also U3.1 (VIN), U3.3 (EN), C1.1, C12.2, D1.1 (K), D7.1 (K), J2.3 (Pin_3)
- net at U2.14 (VINT): now also C13.2
- net AIN2: now reaches U2.15 (AIN2)
- net AIN1: now reaches U2.16 (AIN1)
- net at U2.2 (AOUT1): now also J2.1 (Pin_1)
- net at U2.3 (AISEN): now also R14.1
- net at U2.4 (AOUT2): now also J2.2 (Pin_2)
- net at U2.5 (BOUT2): now also J2.5 (Pin_5)
- net at U2.6 (BISEN): now also R15.1
- net at U2.7 (BOUT1): now also J2.4 (Pin_4)
- net FAULT: now reaches U2.8 (nFAULT)
- net FAULT: now also R18.2
- net BIN1: now reaches U2.9 (BIN1)
- net VCC: now reaches C2.1, FB1.2, USB1.11 (VBUS), USB1.2 (VBUS)
- net VCC: now also D6.4 (VCC)
- net at J1.6 (Pin_6): now also D7.2 (A)
- new net: D2.2 (A), R7.1
- new net: D3.2 (A), R8.1
- new net: D4.2 (A), R9.1
- new net: D5.2 (A), R10.1
- new net SW_Down: R2.2, SW2.2
- new net SW_Mode: R1.2, SW1.2
- new net SW_Up: R4.2, SW3.2
Other:
- moved on the sheet: C2, C3, C5, C6, C7, D6, FB1, R11, R12, R13, R3, R5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

Commit message: pcb placement
Parts:
- added D8: Power, LED_SMD:LED_0603_1608Metric, symbol Device:LED
- added R19, R20, R21: 330, Resistor_SMD:R_0603_1608Metric, symbol Device:R
- J1: footprint (none) -> Connector_PinHeader_2.54mm:PinHeader_2x05_P2.54mm_Horizontal
- J2: footprint (none) -> Connector_PinHeader_2.54mm:PinHeader_1x05_P2.54mm_Vertical
- SW1, SW2, SW3, SW4, SW5: footprint (none) -> Switches_SMD:PTS636_SMT_G
Connections:
- net +3V3: now also R19.2
- net GND: now also D8.1 (K)
- net USART_RX: now also R21.2; no longer U1.14 (PA11)
- net USART_TX: now also R20.2; no longer U1.13 (PA10)
- new net: R20.1, U1.13 (PA10)
- new net: R21.1, U1.14 (PA11)
- new net: D8.2 (A), R19.1
Changed lines of the file:
@@
 Text Label 5250 4800 0    50   ~ 0
 USB_DM
-Text Label 5250 3500 0    50   ~ 0
+Text Label 4850 3500 0    50   ~ 0
 USART_RX
-Text Label 5250 3400 0    50   ~ 0
+Text Label 4850 3400 0    50   ~ 0
 USART_TX
 Wire Wire Line
@@
 Text Label 5250 5700 0    50   ~ 0
 RESET
-Wire Wire Line
-	5250 3400 5850 3400
-Wire Wire Line
-	5250 3500 5850 3500
 $Comp
 L Connector_Generic:Conn_02x05_Odd_Even J1
@@
 F 0 "J1" H 9400 4817 50  0000 C CNN
 F 1 "Conn_02x05_Odd_Even" H 9400 4726 50  0000 C CNN
-F 2 "" H 9350 4400 50  0001 C CNN
+F 2 "Connector_PinHeader_2.54mm:PinHeader_2x05_P2.54mm_Horizontal" H 9350 4400 50  0001 C CNN
 F 3 "~" H 9350 4400 50  0001 C CNN
 	1    9350 4400
@@
 F 0 "SW5" V 4346 5852 50  0000 R CNN
 F 1 "Reset" V 4255 5852 50  0000 R CNN
-F 2 "" H 4300 6100 50  0001 C CNN
+F 2 "Switches_SMD:PTS636_SMT_G" H 4300 6100 50  0001 C CNN
 F 3 "~" H 4300 6100 50  0001 C CNN
 	1    4300 5900
@@
 F 0 "J2" H 10880 2592 50  0000 L CNN
 F 1 "Conn_01x05" H 10880 2501 50  0000 L CNN
-F 2 "" H 10800 2550 50  0001 C CNN
+F 2 "Connector_PinHeader_2.54mm:PinHeader_1x05_P2.54mm_Vertical" H 10800 2550 50  0001 C CNN
 F 3 "~" H 10800 2550 50  0001 C CNN
 	1    10800 2550
@@
 F 0 "SW1" H 1300 4235 50  0000 C CNN
 F 1 "Mode" H 1300 4144 50  0000 C CNN
-F 2 "" H 1300 4150 50  0001 C CNN
+F 2 "Switches_SMD:PTS636_SMT_G" H 1300 4150 50  0001 C CNN
 F 3 "~" H 1300 4150 50  0001 C CNN
 	1    1300 3950
@@
 F 0 "SW2" H 1300 4585 50  0000 C CNN
 F 1 "Up" H 1300 4494 50  0000 C CNN
-F 2 "" H 1300 4500 50  0001 C CNN
+F 2 "Switches_SMD:PTS636_SMT_G" H 1300 4500 50  0001 C CNN
 F 3 "~" H 1300 4500 50  0001 C CNN
 	1    1300 4300
@@
 F 0 "SW3" H 1300 4935 50  0000 C CNN
 F 1 "Down" H 1300 4844 50  0000 C CNN
-F 2 "" H 1300 4850 50  0001 C CNN
+F 2 "Switches_SMD:PTS636_SMT_G" H 1300 4850 50  0001 C CNN
 F 3 "~" H 1300 4850 50  0001 C CNN
 	1    1300 4650
@@
 F 0 "SW4" H 1300 5285 50  0000 C CNN
 F 1 "Sel" H 1300 5194 50  0000 C CNN
-F 2 "" H 1300 5200 50  0001 C CNN
+F 2 "Switches_SMD:PTS636_SMT_G" H 1300 5200 50  0001 C CNN
 F 3 "~" H 1300 5200 50  0001 C CNN
 	1    1300 5000
@@
 Wire Wire Line
 	5550 3900 5850 3900
+$Comp
+L Device:R R20
+U 1 1 608C7709
+P 5650 3400
+F 0 "R20" V 5550 3250 50  0000 C CNN
+F 1 "330" V 5650 3400 50  0000 C CNN
+F 2 "Resistor_SMD:R_0603_1608Metric" V 5580 3400 50  0001 C CNN
+F 3 "~" H 5650 3400 50  0001 C CNN
+	1    5650 3400
+	0    1    1    0
+$EndComp
+$Comp
+L Device:R R21
+U 1 1 608CE78D
+P 5650 3500
+F 0 "R21" V 5750 3350 50  0000 C CNN
+F 1 "330" V 5650 3500 50  0000 C CNN
+F 2 "Resistor_SMD:R_0603_1608Metric" V 5580 3500 50  0001 C CNN
+F 3 "~" H 5650 3500 50  0001 C CNN
+	1    5650 3500
+	0    1    1    0
+$EndComp
+Wire Wire Line
+	4850 3400 5500 3400
+Wire Wire Line
+	4850 3500 5500 3500
+Wire Wire Line
+	5800 3400 5850 3400
+Wire Wire Line
+	5800 3500 5850 3500
+$Comp
+L Device:LED D8
+U 1 1 608F55EC
+P 2900 5700
+F 0 "D8" H 3100 5650 50  0000 C CNN
+F 1 "Power" H 2750 5800 50  0000 C CNN
+F 2 "LED_SMD:LED_0603_1608Metric" H 2900 5700 50  0001 C CNN
+F 3 "~" H 2900 5700 50  0001 C CNN
+	1    2900 5700
+	-1   0    0    1
+$EndComp
+$Comp
+L Device:R R19
+U 1 1 608F55F2
+P 2450 5700
+F 0 "R19" V 2243 5700 50  0000 C CNN
+F 1 "330" V 2334 5700 50  0000 C CNN
+F 2 "Resistor_SMD:R_0603_1608Metric" V 2380 5700 50  0001 C CNN
+F 3 "~" H 2450 5700 50  0001 C CNN
+	1    2450 5700
+	0    1    1    0
+$EndComp
+Wire Wire Line
+	2600 5700 2750 5700
+Wire Wire Line
+	2300 5700 2150 5700
+Wire Wire Line
+	2150 5700 2150 5500
+Connection ~ 2150 5500
+$Comp
+L power:GND #PWR0145
+U 1 1 6090537D
+P 3200 5700
+F 0 "#PWR0145" H 3200 5450 50  0001 C CNN
+F 1 "GND" H 3205 5527 50  0000 C CNN
+F 2 "" H 3200 5700 50  0001 C CNN
+F 3 "" H 3200 5700 50  0001 C CNN
+	1    3200 5700
+	1    0    0    -1
+$EndComp
+Wire Wire Line
+	3050 5700 3200 5700
 $EndSCHEMATC

Commit message: connections
Parts:
- added R22: 10k, Resistor_SMD:R_0603_1608Metric, symbol Device:R
Connections:
- net AIN1: now also U1.19 (PA18)
- net AIN2: now also U1.20 (PA19)
- net BIN1: now also U1.21 (PA22)
- net BIN2: now also U1.22 (PA23)
- net FAULT: now also U1.25 (PA27)
- net GND: now also R22.2
- net SW_Down: now also U1.15 (PA14)
- net SW_Mode: now also U1.12 (PA09)
- net SW_Up: now also U1.17 (PA16)
- net nSleep: now also U1.18 (PA17), R22.1
- net at U1.3 (PA02): now also D2.1 (K)
- net at U1.4 (PA03): now also D3.1 (K)
- net at U1.5 (PA04): now also D4.1 (K)
- net at U1.6 (PA05): now also D5.1 (K)
- no-connect marks 0 -> 6
Other:
- moved on the sheet: C5, C6, D2, D3, D4, D5, D8, R10, R19, R7, R8, R9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

Commit message: added con for Sel, added gerber
Parts:
- added J3: Conn_01x02, Connector_PinHeader_2.54mm:PinHeader_1x02_P2.54mm_Vertical, symbol Connector_Generic:Conn_01x02
- H1, H2, H3, H4: footprint MountingHole:MountingHole_3.2mm_M3_DIN965 -> MountingHole:MountingHole_3.2mm_M3_DIN965_Pad; symbol Mechanical:MountingHole -> Mechanical:MountingHole_Pad
Connections:
- net BIN1: now also U1.22 (PA23); no longer U1.21 (PA22)
- net BIN2: now also U1.21 (PA22); no longer U1.22 (PA23)
- net GND: now also H1.1, H2.1, H3.1, H4.1, J3.1 (Pin_1)
- net SW_Sel: now also J3.2 (Pin_2)
- net A1: now reaches U2.2 (AOUT1)
- net A1: now also J2.5 (Pin_5); no longer J2.1 (Pin_1)
- net A2: now reaches U2.4 (AOUT2)
- net A2: now also J2.4 (Pin_4); no longer J2.2 (Pin_2)
- net B2: now reaches U2.5 (BOUT2)
- net B2: now also J2.2 (Pin_2); no longer J2.5 (Pin_5)
- net B1: now reaches U2.7 (BOUT1)
- net B1: now also J2.1 (Pin_1); no longer J2.4 (Pin_4)
- net _DM: now reaches R11.2, USB1.5 (DN2), USB1.7 (DN1)
- net _DM: now also D6.3 (I/O2)
- net _DP: now reaches R12.2, USB1.6 (DP1), USB1.8 (DP2)
- net _DP: now also D6.2 (I/O1)
Other:
- note added: "StepperControl RevA"
- moved on the sheet: J2
